File: hardware/ssr_24v_by4/ssr_24v_by4.kicad_pcb (KiCad board)
At the start: 2 copper layers, 65 x 90 mm, 45 parts, among them J1 1190297, J2 1190297, J3 1190297, J4 1190297, Q1 IRF4905PBF, Q2 IRF4905PBF, Q3 IRF4905PBF, Q4 IRF4905PBF

Commit message: README link fixes and WIP PCB etc.
Parts:
- added #LOGO_CC1: Symbol_CreativeCommons_SilkScreenTop_Type2_Big, Symbol:Symbol_CreativeCommons_SilkScreenTop_Type2_Big, F.Cu at (50.0, 71.0)
- added #LOGO_OSHW1: OSHW-Logo_11.4x12mm_SilkScreen, Symbol:OSHW-Logo_11.4x12mm_SilkScreen, F.Cu at (54.0, 52.8)
- added FID1: Fiducial, Fiducial:Fiducial_0.5mm_Mask1mm, F.Cu at (20.5, 28.5)
- added FID2: Fiducial, Fiducial:Fiducial_0.5mm_Mask1mm, F.Cu at (75.5, 28.5)
- added FID3: Fiducial, Fiducial:Fiducial_0.5mm_Mask1mm, F.Cu at (75.5, 90.5)
- HQ1, HQ2, HQ3, HQ4: footprint MountingHole:MountingHole_3.2mm_M3_Pad_Via -> dragon_mobile:MountingHole_6.1mm_Pad_Via
- moved TVSP2 0.15 mm to (27.7, 37.5)
Routing:
- net /a2: track 45.5 -> 41.9 mm
- net OUT3: track 62.1 -> 63.3 mm, vias 0 -> 8
- net OUT4: vias 0 -> 8
- net OUT2: vias 0 -> 8
- net OUT1: vias 0 -> 8
- net +BATT: vias 75 -> 106
Other:
- board text added: "Rev: 0.0.2"
- board text added: "© 2022 Michael Cummings"
