File: hardware/ssr_24v_by4/ssr_24v_by4.kicad_sch (KiCad schematic)
At the start: 45 parts, among them J1 1190297, J2 1190297, J3 1190297, J4 1190297, Q1 IRF4905PBF, Q2 IRF4905PBF, Q3 IRF4905PBF, Q4 IRF4905PBF

Commit message: README link fixes and WIP PCB etc.
Parts:
- added FID1, FID2, FID3: Fiducial, Fiducial:Fiducial_0.5mm_Mask1mm, symbol Mechanical:Fiducial
- HQ1, HQ3: value HeatsinkHole -> Access Hole; footprint MountingHole:MountingHole_3.2mm_M3_Pad_Via -> dragon_mobile:MountingHole_6.1mm_Pad_Via; Package (none) -> Other; Type (none) -> THT; now in the parts list
- HQ2, HQ4: value HeatsinkHole -> Access Hole; footprint MountingHole:MountingHole_3.2mm_M3_Pad_Via -> dragon_mobile:MountingHole_6.1mm_Pad_Via; Package (none) -> Other; Type (none) -> THT
Other:
- note added: "Fiducials"
- note added: "MOSFET Mounting Access Holes"
- note added: "WARNING: Q1-8 mounting tabs are at +BATT voltage and MUST BE electrically isolated from any grounded heatsinks."
- note removed: "MOSFET Mounting Holes/Access"
